Commit message: Use the standard ros_gazebo and switch back urdf
Switch back URDF to what it was so it works with RVIZ and gazebo. Also
use ros_gazebo instead of ign_gazebo since it might work better with
moveit and you can use GPU acceleration on WSL.

File: preliminary-simulation/models/lleap_exo.urdf.xacro (robot description, xacro)
@@ -31,5 +31,5 @@
   <!-- secure (fix) model in Gazebo: world <> link0 = fixed base_link = torso -->
   <joint name="global_fixed" type="fixed">
-    <origin xyz="0 0 1" rpy="0 0 ${pi}" /> <!--changed z component so robot isnt stuck in ground -->
+    <origin xyz="0 0 0" rpy="0 0 ${pi}" />
     <parent link="world"/>
     <child link="base_link"/>
@@ -79,5 +79,5 @@
         <origin xyz="0 0 0" rpy="0 0 0" />
         <geometry>
-          <mesh filename="$(find preliminary-simulation)/meshes/hip_base.STL" />
+          <mesh filename="package://preliminary-simulation/meshes/${link0}.STL" />
         </geometry>
         <material name="">
@@ -88,5 +88,5 @@
         <origin xyz="0 0 0" rpy="0 0 0" />
         <geometry>
-          <mesh filename="$(find preliminary-simulation)/meshes/hip_base.STL" />
+          <mesh filename="package://preliminary-simulation/meshes/${link0}.STL" />
         </geometry>
       </collision>
@@ -117,5 +117,5 @@
         <origin xyz="0 0 0" rpy="${pi / 2} 0 ${-(180 - 12) * pi / 180}" />
         <geometry>
-          <mesh filename="$(find preliminary-simulation)/meshes/thigh.STL" />
+          <mesh filename="package://preliminary-simulation/meshes/${link1}.STL" />
         </geometry>
         <material name="">
@@ -126,5 +126,5 @@
         <origin xyz="0 0 0" rpy="${pi / 2} 0 ${-(180 - 12) * pi / 180}" />
         <geometry>
-          <mesh filename="$(find preliminary-simulation)/meshes/thigh.STL" />
+          <mesh filename="package://preliminary-simulation/meshes/${link1}.STL" />
         </geometry>
       </collision>
@@ -154,5 +154,5 @@
         <origin xyz="0 0 0" rpy="${pi / 2} 0 ${-(180 - 34) * pi / 180}" />
         <geometry>
-          <mesh filename="$(find preliminary-simulation)/meshes/shank.STL" />
+          <mesh filename="package://preliminary-simulation/meshes/${link2}.STL" />
         </geometry>
         <material name="">
@@ -163,5 +163,5 @@
         <origin xyz="0 0 0" rpy="${pi / 2} 0 ${-(180 - 34) * pi / 180}" />
         <geometry>
-          <mesh filename="$(find preliminary-simulation)/meshes/shank.STL" />
+          <mesh filename="package://preliminary-simulation/meshes/${link2}.STL" />
         </geometry>
       </collision>
